File: C11.kicad_pcb (KiCad board)
At the start: 2 copper layers, 160.3 x 71.7 mm, 166 parts, among them IC1 MPM3610AGQV-P, IC2 THVD1450DRBR, IC3 THVD1450DRBR, IC4 THVD1450DRBR, IC5 THVD1450DRBR, IC6 MAX17613AATP+, IC8 MAX17613AATP+, J1 V24, J2 UDPI, J21 Conn_01x16, J22 RTBUS.out, J23 RTBUS.in, J3 Slot-0, J4 Slot-a1, J5 UDPI, J6 Screw_Terminal_01x04, J7 Slot-a0, J8 Screw_Terminal_01x02, J9 Conn_01x06, Q1 IRLML2060, U1 ATmega4809-M, U3 74AHC1G02, U4 74AHC1G02, U5 L78M12, U7 INA181A4, U9 ATmega4809-A, X1 ASE-24MHz

Commit message: Initial commit
Parts:
- IC1: footprint _Samac:MPM3610AGQVP -> RTB_foot:MPM3610AGQVP
- IC2, IC3, IC4, IC5: footprint _Samac:SON65P300X300X100-9N-D -> RTB_foot:SON65P300X300X100-9N-D
Connections:
- IC6 pad 14: Vbst.0 -> (no net)
- IC6 pad 2: Vsrc -> (no net)
- IC8 pad 14: Vbst.1 -> (no net)
- IC8 pad 2: Vsrc -> (no net)

Commit message: Initial commit
Parts:
- IC1: footprint RTB_foot:MPM3610AGQVP -> RTB:MPM3610AGQVP
- IC2, IC3, IC4, IC5: footprint RTB_foot:SON65P300X300X100-9N-D -> RTB:SON65P300X300X100-9N-D
